File: eByteAdapter.kicad_pcb (KiCad board)
At the start: 2 copper layers, 17.2 x 19.6 mm, 2 parts, among them J1 eByte, J2 CC1101 Module

Commit message: update
Parts:
- moved J1 0.50 mm to (28.5, 35.0)
Changed lines of the file:
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@@
     (thickness 1.6)
     (drawings 18)
-    (tracks 38)
+    (tracks 42)
     (zones 0)
     (modules 2)
@@
   )
   (module Connector_PinHeader_1.27mm:PinHeader_1x08_P1.27mm_Vertical (layer F.Cu)
-    (at 28 35 90)
+    (at 28.5 35 90)
     (descr "Through hole straight pin header, 1x08, 1.27mm pitch, single row")
     (tags "Through hole pin header THT 1x08 1.27mm single row")
@@
   (via (at 32.5 25) (size 0.8) (drill 0.4) (layers F.Cu B.Cu) (net 1))
   (via (at 37.5 25) (size 0.8) (drill 0.4) (layers F.Cu B.Cu) (net 1))
-  (segment (start 35.62 35) (end 36.9 36.2) (width 0.25) (layer B.Cu) (net 2))
   (segment (start 36.9 36.2) (end 38 37) (width 0.25) (layer B.Cu) (net 2))
+  (segment (start 36.1 35) (end 36.9 36.2) (width 0.25) (layer B.Cu) (net 2))
   (segment (start 34.8253 35.8253) (end 36 37) (width 0.25) (layer F.Cu) (net 3))
-  (segment (start 34.35 35) (end 34.35 35.8253) (width 0.25) (layer F.Cu) (net 3))
-  (segment (start 34.35 35.8253) (end 34.8253 35.8253) (width 0.25) (layer F.Cu) (net 3))
+  (segment (start 34.8253 35.8253) (end 34.8253 35.0253) (width 0.25) (layer F.Cu) (net 3))
+  (segment (start 34.8253 35.0253) (end 34.8 35) (width 0.25) (layer F.Cu) (net 3))
   (segment (start 32 37) (end 32 35.9997) (width 0.25) (layer B.Cu) (net 4))
-  (segment (start 33.08 35) (end 32.0803 35.9997) (width 0.25) (layer B.Cu) (net 4))
   (segment (start 32.0803 35.9997) (end 32 35.9997) (width 0.25) (layer B.Cu) (net 4))
-  (segment (start 31.81 35) (end 33.81 37) (width 0.25) (layer F.Cu) (net 5))
+  (segment (start 32.0803 35.9997) (end 32.6003 35.9997) (width 0.25) (layer B.Cu) (net 4))
+  (segment (start 32.6003 35.9997) (end 33.5 35.1) (width 0.25) (layer B.Cu) (net 4))
+  (segment (start 33.5 35.1) (end 33.5 35) (width 0.25) (layer B.Cu) (net 4))
   (segment (start 33.81 37) (end 34 37) (width 0.25) (layer F.Cu) (net 5))
-  (segment (start 38.413 35.5297) (end 40.5297 35.5297) (width 0.25) (layer B.Cu) (net 6))
-  (segment (start 40.5297 35.5297) (end 42 37) (width 0.25) (layer B.Cu) (net 6))
-  (segment (start 30.54 35) (end 31.3696 34.1704) (width 0.25) (layer F.Cu) (net 6))
-  (segment (start 31.3696 34.1704) (end 37.265 34.1704) (width 0.25) (layer F.Cu) (net 6))
-  (segment (start 37.265 34.1704) (end 38.413 35.3184) (width 0.25) (layer F.Cu) (net 6))
-  (segment (start 38.413 35.3184) (end 38.413 35.5297) (width 0.25) (layer F.Cu) (net 6))
-  (via (at 38.413 35.5297) (size 0.8) (layers F.Cu B.Cu) (net 6))
-  (segment (start 40 35.9997) (end 37.7204 33.7201) (width 0.25) (layer F.Cu) (net 7))
-  (segment (start 37.7204 33.7201) (end 30.5499 33.7201) (width 0.25) (layer F.Cu) (net 7))
-  (segment (start 30.5499 33.7201) (end 29.27 35) (width 0.25) (layer F.Cu) (net 7))
+  (segment (start 32.3 35) (end 33.81 37) (width 0.25) (layer F.Cu) (net 5))
+  (segment (start 40.6 35.5) (end 42 37) (width 0.25) (layer B.Cu) (net 6))
+  (segment (start 38.7 35.5) (end 40.6 35.5) (width 0.25) (layer B.Cu) (net 6))
+  (segment (start 38.300001 35.100001) (end 38.7 35.5) (width 0.25) (layer F.Cu) (net 6))
+  (via (at 38.7 35.5) (size 0.8) (drill 0.4) (layers F.Cu B.Cu) (net 6))
+  (segment (start 38.300001 34.688999) (end 38.300001 35.100001) (width 0.25) (layer F.Cu) (net 6))
+  (segment (start 37.781402 34.1704) (end 38.300001 34.688999) (width 0.25) (layer F.Cu) (net 6))
+  (segment (start 31.3696 34.1704) (end 37.781402 34.1704) (width 0.25) (layer F.Cu) (net 6))
+  (segment (start 31 35) (end 31.3696 34.1704) (width 0.25) (layer F.Cu) (net 6))
+  (segment (start 30.5499 33.7201) (end 29.7 35) (width 0.25) (layer F.Cu) (net 7))
+  (segment (start 38.3 33.7) (end 30.5499 33.7201) (width 0.25) (layer F.Cu) (net 7))
+  (segment (start 40 35.9997) (end 38.3 33.7) (width 0.25) (layer F.Cu) (net 7))
   (segment (start 40 37) (end 40 35.9997) (width 0.25) (layer F.Cu) (net 7))
-  (segment (start 28 35) (end 28 37) (width 0.25) (layer F.Cu) (net 8))
+  (segment (start 28 35.5) (end 28 37) (width 0.25) (layer F.Cu) (net 8))
+  (segment (start 28.5 35) (end 28 35.5) (width 0.25) (layer F.Cu) (net 8))
   (zone (net 1) (net_name /GND) (layer B.Cu) (hatch edge 0.508)
     (connect_pads (clearance 0.508))

Commit message: update kicad
Other:
- net class Default removed
